File: board_down.kicad_pcb (KiCad board)
At the start: 2 copper layers, 98 x 98 mm, 17 parts, among them J101 Power Sw 1 Bridge, J102 Power Sw 2 Bridge, J103 Battery+ Socket, J104 Battery- Socket, J116 5V Bridge, J117 3.3V Bridge, J118 LRC Bridge, J119 BCLK Bridge, J120 DIN Bridge, U101 MT3608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

Commit message: checkpoint
Parts:
- moved C103 2.84 mm to (9.01, 62.2)
Routing:
- net GND: track 192.9 -> 198.1 mm
- net Net-(D102-A): track 25.7 -> 23.4 mm
Changed lines of the file:
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@@
   )
   (footprint "Capacitor_THT:CP_Radial_D18.0mm_P7.50mm" (layer "F.Cu")
-    (at 11.55 63.5)
+    (at 9.01 62.23)
     (descr "CP, Radial series, Radial, pin pitch=7.50mm, , diameter=18mm, Electrolytic Capacitor")
     (tags "CP Radial series Radial pin pitch 7.50mm  diameter 18mm Electrolytic Capacitor")
@@
     )
   )
+  (gr_circle (center 12.7 62.07) (end 22.2 62.07)
+    (stroke (width 0.15) (type default)) (fill none) (layer "F.SilkS"))
   (gr_line (start 73.96 7.095) (end 73.46 7.961)
     (stroke (width 0.15) (type default)) (layer "Edge.Cuts"))
@@
   (segment (start 36.83 91.44) (end 33.02 87.63) (width 1) (layer "F.Cu") (net 2))
   (segment (start 49.53 91.44) (end 36.83 91.44) (width 1) (layer "F.Cu") (net 2))
+  (segment (start 33.02 48.26) (end 33.02 78.74) (width 1) (layer "F.Cu") (net 2))
   (segment (start 33.02 36.83) (end 33.02 31.75) (width 1) (layer "F.Cu") (net 2))
-  (segment (start 22.86 63.5) (end 33.02 73.66) (width 1) (layer "B.Cu") (net 2))
-  (segment (start 33.02 48.26) (end 33.02 78.74) (width 1) (layer "B.Cu") (net 2))
-  (segment (start 22.86 63.5) (end 19.05 63.5) (width 1) (layer "B.Cu") (net 2))
+  (segment (start 16.51 62.23) (end 33.02 78.74) (width 1) (layer "B.Cu") (net 2))
   (segment (start 7.625 44.45) (end 6.35 44.45) (width 1) (layer "F.Cu") (net 3))
+  (segment (start 2.54 55.88) (end 2.54 48.26) (width 1) (layer "F.Cu") (net 3))
   (segment (start 6.35 44.45) (end 2.54 48.26) (width 1) (layer "F.Cu") (net 3))
-  (segment (start 11.43 63.5) (end 2.54 54.61) (width 1) (layer "F.Cu") (net 3))
-  (segment (start 11.55 63.5) (end 11.43 63.5) (width 1) (layer "F.Cu") (net 3))
-  (segment (start 2.54 54.61) (end 2.54 48.26) (width 1) (layer "F.Cu") (net 3))
+  (segment (start 8.89 62.23) (end 2.54 55.88) (width 1) (layer "F.Cu") (net 3))
+  (segment (start 9.01 62.23) (end 8.89 62.23) (width 1) (layer "F.Cu") (net 3))
   (segment (start 10.16 48.26) (end 12.695 48.26) (width 1) (layer "F.Cu") (net 4))
   (segment (start 16.51 44.45) (end 15.245 44.45) (width 1) (layer "F.Cu") (net 5))

Commit message: checkpoint
Parts:
- J101, J102, J103, J104, J116, J117, J118, J119, J120: footprint MyPinSocket:MyPinSocket -> Connector_PinSocket_2.54mm:PinSocket_1x01_P2.54mm_Vertical
